Commit message: updated mecanum URDF

File: src/urdf/roboost_mecanum_robot.urdf.xacro (robot description, xacro)
@@ -1,5 +1,5 @@
 <?xml version="1.0"?>
 <robot xmlns:xacro="http://www.ros.org/wiki/xacro"  name="roboost_mecanum_robot">
-    <xacro:include filename="roboost_materials.xacro"/>
+    <xacro:include filename="res/roboost_materials.xacro"/>
     <!-- TODO: determine values -->
     <xacro:property name="chassis_length" value="0.42"/>
@@ -14,6 +14,6 @@
     <xacro:property name="wheelbase" value="0.38"/>
     <xacro:property name="track" value="0.32"/>
-    <link name="world"></link>
-    <link name="chassis_link">
+    <!--link name="world"></link-->
+    <link name="base_link">
         <visual>
             <geometry>
@@ -115,11 +115,31 @@
         </inertial>
     </link>
-    <joint name="world_to_chassis_joint" type="fixed">
+    <link name="lidar_link">
+        <visual>
+            <geometry>
+                <cylinder radius="0.05" length="0.05"/>
+            </geometry>
+            <origin xyz="0.0 0.0 0.0" rpy="0.0 0.0 0.0"/>
+            <material name="grey"/>
+        </visual>
+        <collision>
+            <geometry>
+                <cylinder radius="0.05" length="0.05"/>
+            </geometry>
+            <origin xyz="0.0 0.0 0.0" rpy="0.0 0.0 0.0"/>
+        </collision>
+        <inertial>
+            <mass value="1.0"/>
+            <origin xyz="0.0 0.0 0.0" rpy="0.0 0.0 0.0"/>
+            <inertia ixx="0.1" ixy="0.0" ixz="0.0" iyy="0.1" iyz="0.0" izz="0.1"/>
+        </inertial>
+    </link>
+    <!--joint name="world_to_chassis_joint" type="fixed">
         <parent link="world"/>
-        <child link="chassis_link"/>
+        <child link="base_link"/>
         <origin xyz="0.0 0.0 0.0" rpy="0.0 0.0 0.0"/>
-    </joint>
+    </joint-->
     <joint name="wheel_front_left_joint" type="continuous">
-        <parent link="chassis_link"/>
+        <parent link="base_link"/>
         <child link="wheel_front_left_link"/>
         <origin xyz="${wheelbase / 2} ${track / 2} 0.0" rpy="${pi * 3 / 2} 0.0 0.0"/>
@@ -128,5 +148,5 @@
     </joint>
     <joint name="wheel_front_right_joint" type="continuous">
-        <parent link="chassis_link"/>
+        <parent link="base_link"/>
         <child link="wheel_front_right_link"/>
         <origin xyz="${wheelbase / 2} -${track / 2} 0.0" rpy="${pi / 2} 0.0 0.0"/>
@@ -135,5 +155,5 @@
     </joint>
     <joint name="wheel_back_left_joint" type="continuous">
-        <parent link="chassis_link"/>
+        <parent link="base_link"/>
         <child link="wheel_back_left_link"/>
         <origin xyz="-${wheelbase / 2} ${track / 2} 0.0" rpy="${pi * 3 / 2} 0.0 0.0"/>
@@ -142,5 +162,5 @@
     </joint>
     <joint name="wheel_back_right_joint" type="continuous">
-        <parent link="chassis_link"/>
+        <parent link="base_link"/>
         <child link="wheel_back_right_link"/>
         <origin xyz="-${wheelbase / 2} -${track / 2} 0.0" rpy="${pi / 2} 0.0 0.0"/>
@@ -148,3 +168,8 @@
         <limit effort="1000.0" velocity="1000.0"/>
     </joint>
+    <joint name="lidar_joint" type="fixed">
+        <parent link="base_link"/>
+        <child link="lidar_link"/>
+        <origin xyz="0.0 0.0 ${chassis_height}" rpy="${pi} 0.0 ${pi * 3 / 2}"/>
+    </joint>
 </robot>
