Commit message: added curesed meshes

File: src/tf_broadcast_package/urdf/roboost_materials.xacro (robot description, xacro)
@@ -13,3 +13,18 @@
         <color rgba="0 0 1 1"/>
     </material>
+    <material name="red">
+        <color rgba="1 0 0 1"/>
+    </material>
+    <material name="green">
+        <color rgba="0 1 0 1"/>
+    </material>
+    <material name="yellow">
+        <color rgba="1 1 0 1"/>
+    </material>
+    <material name="black">
+        <color rgba="0 0 0 1"/>
+    </material>
+    <material name="purple">
+        <color rgba="0.5 0 0.5 1"/>
+    </material>
 </robot>

File: src/tf_broadcast_package/urdf/roboost_mecanum_robot.urdf.xacro (robot description, xacro)
@@ -18,7 +18,7 @@
         <visual>
             <geometry>
-                <box size="${chassis_length} ${chassis_width} ${chassis_height}"/>
-            </geometry>
-            <origin xyz="0 0 0.05" rpy="0.0 0.0 0.0"/>
+                <mesh filename="file:///home/geibinger/Projects/Roboost/Roboost-Cerebrum/src/tf_broadcast_package/meshes/Chassis.STL" scale="0.001 0.001 0.001"/>
+            </geometry>
+            <origin xyz="0 0 0.05" rpy="${pi / 2} 0.0 0.0"/>
             <material name="orange"/>
         </visual>
@@ -38,5 +38,6 @@
         <visual>
             <geometry>
-                <cylinder radius="${wheel_radius}" length="${wheel_width}"/>
+                <!--cylinder radius="${wheel_radius}" length="${wheel_width}"/-->
+                <mesh filename="file:///home/geibinger/Projects/Roboost/Roboost-Cerebrum/src/tf_broadcast_package/meshes/Mecanum-Wheel-Left.STL" scale="0.001 0.001 0.001"/>
             </geometry>
             <origin xyz="0.0 0.0 0.03" rpy="0.0 0.0 0.0"/>
@@ -121,5 +122,5 @@
             </geometry>
             <origin xyz="0.0 0.0 0.0" rpy="0.0 0.0 0.0"/>
-            <material name="grey"/>
+            <material name="red"/>
         </visual>
         <collision>
@@ -133,4 +134,45 @@
             <origin xyz="0.0 0.0 0.0" rpy="0.0 0.0 0.0"/>
             <inertia ixx="0.1" ixy="0.0" ixz="0.0" iyy="0.1" iyz="0.0" izz="0.1"/>
+        </inertial>
+    </link>
+    <link name="camera_link">
+        <visual>
+            <geometry>
+                <cylinder radius="0.01" length="0.02"/>
+                <box size="0.02 0.02 0.01"/>
+            </geometry>
+            <origin xyz="0.0 0.0 0.0" rpy="0.0 0.0 0.0"/>
+            <material name="purple"/>
+        </visual>
+        <collision>
+            <geometry>
+                <box size="0.02 0.02 0.02"/>
+            </geometry>
+            <origin xyz="0.0 0.0 0.0" rpy="0.0 0.0 0.0"/>
+        </collision>
+        <inertial>
+            <mass value="1.0"/>
+            <origin xyz="0.0 0.0 0.0" rpy="0.0 0.0 0.0"/>
+            <inertia ixx="0.01" ixy="0.0" ixz="0.0" iyy="0.01" iyz="0.0" izz="0.01"/>
+        </inertial>
+    </link>
+    <link name="imu">
+        <visual>
+            <geometry>
+                <box size="0.02 0.02 0.01"/>
+            </geometry>
+            <origin xyz="0.0 0.0 0.0" rpy="0.0 0.0 0.0"/>
+            <material name="blue"/>
+        </visual>
+        <collision>
+            <geometry>
+                <box size="0.02 0.02 0.01"/>
+            </geometry>
+            <origin xyz="0.0 0.0 0.0" rpy="0.0 0.0 0.0"/>
+        </collision>
+        <inertial>
+            <mass value="1.0"/>
+            <origin xyz="0.0 0.0 0.0" rpy="0.0 0.0 0.0"/>
+            <inertia ixx="0.01" ixy="0.0" ixz="0.0" iyy="0.01" iyz="0.0" izz="0.01"/>
         </inertial>
     </link>
@@ -171,5 +213,15 @@
         <parent link="base_link"/>
         <child link="lidar_link"/>
-        <origin xyz="0.0 0.0 ${chassis_height}" rpy="${pi} 0.0 ${pi * 3 / 2}"/>
+        <origin xyz="0.0 -0.05 ${chassis_height}" rpy="${pi} 0.0 ${pi * 3 / 2}"/>
+    </joint>
+    <joint name="camera_joint" type="fixed">
+        <parent link="base_link"/>
+        <child link="camera_link"/>
+        <origin xyz="${-chassis_length / 2} 0.08 ${chassis_height -0.05}" rpy="0.0 ${pi * 3 / 2} 0.0"/>
+    </joint>
+    <joint name="imu_joint" type="fixed">
+        <parent link="base_link"/>
+        <child link="imu"/>
+        <origin xyz="${-chassis_length / 2 + 0.05} 0.08 ${chassis_height -0.015}" rpy="0.0 0.0 0.0"/>
     </joint>
 </robot>
