Commit message: added relative paths, updated STL files

File: src/tf_broadcast_package/urdf/roboost_mecanum_robot.urdf.xacro (robot description, xacro)
@@ -5,20 +5,20 @@
     <xacro:property name="chassis_length" value="0.42"/>
     <xacro:property name="chassis_width" value="0.28"/>
-    <xacro:property name="chassis_height" value="0.14"/>
+    <xacro:property name="chassis_height" value="0.108"/> <!-- ! Measured from wheel axis to top plate -->
     <xacro:property name="chassis_mass" value="20.0"/>
     <xacro:property name="chassis_inertia" value="4.0"/>
-    <xacro:property name="wheel_radius" value="0.075"/>
+    <xacro:property name="wheel_radius" value="0.0835"/>
     <xacro:property name="wheel_width" value="0.05"/>
     <xacro:property name="wheel_mass" value="1.0"/>
     <xacro:property name="wheel_inertia" value="0.1"/>
-    <xacro:property name="wheelbase" value="0.38"/>
-    <xacro:property name="track" value="0.32"/>
-    <!--link name="world"></link-->
+    <xacro:property name="lidar_height" value="0.0575"/>
+    <xacro:property name="wheelbase" value="0.3185"/>
+    <xacro:property name="track" value="0.38"/>
     <link name="base_link">
         <visual>
             <geometry>
-                <mesh filename="file:///home/geibinger/Projects/Roboost/Roboost-Cerebrum/src/tf_broadcast_package/meshes/Chassis.STL" scale="0.001 0.001 0.001"/>
-            </geometry>
-            <origin xyz="0 0 0.05" rpy="${pi / 2} 0.0 0.0"/>
+                <mesh filename="file://$(find tf_broadcast_package)/meshes/Chassis.STL" scale="0.001 0.001 0.001"/>
+            </geometry>
+            <origin xyz="0.0 0.0 0.0" rpy="${pi / 2} 0.0 0.0"/>
             <material name="orange"/>
         </visual>
@@ -39,14 +39,14 @@
             <geometry>
                 <!--cylinder radius="${wheel_radius}" length="${wheel_width}"/-->
-                <mesh filename="file:///home/geibinger/Projects/Roboost/Roboost-Cerebrum/src/tf_broadcast_package/meshes/Mecanum-Wheel-Left.STL" scale="0.001 0.001 0.001"/>
-            </geometry>
-            <origin xyz="0.0 0.0 0.03" rpy="0.0 0.0 0.0"/>
-            <material name="grey"/>
-        </visual>
-        <collision>
-            <geometry>
-                <cylinder radius="${wheel_radius}" length="${wheel_width}"/>
-            </geometry>
-            <origin xyz="0.0 0.0 0.03" rpy="0.0 0.0 0.0"/>
+                <mesh filename="file://$(find tf_broadcast_package)/meshes/Mecanum-Wheel-Left.STL" scale="0.001 0.001 0.001"/>
+            </geometry>
+            <origin xyz="-${wheel_radius} ${wheel_radius} ${wheel_width}" rpy="${pi} 0.0 0.0"/>
+            <material name="grey"/>
+        </visual>
+        <collision>
+            <geometry>
+                <cylinder radius="${wheel_radius}" length="${wheel_width}"/>
+            </geometry>
+            <origin xyz="0.0 0.0 0.0" rpy="0.0 0.0 0.0"/>
         </collision>
         <inertial>
@@ -59,14 +59,15 @@
         <visual>
             <geometry>
-                <cylinder radius="${wheel_radius}" length="${wheel_width}"/>
-            </geometry>
-            <origin xyz="0.0 0.0 0.03" rpy="0.0 0.0 0.0"/>
-            <material name="grey"/>
-        </visual>
-        <collision>
-            <geometry>
-                <cylinder radius="${wheel_radius}" length="${wheel_width}"/>
-            </geometry>
-            <origin xyz="0.0 0.0 0.03" rpy="0.0 0.0 0.0"/>
+                <!--cylinder radius="${wheel_radius}" length="${wheel_width}"/-->
+                <mesh filename="file://$(find tf_broadcast_package)/meshes/Mecanum-Wheel-Right.STL" scale="0.001 0.001 0.001"/>
+            </geometry>
+            <origin xyz="0.0 0.0 0.0" rpy="0.0 0.0 0.0"/>
+            <material name="grey"/>
+        </visual>
+        <collision>
+            <geometry>
+                <cylinder radius="${wheel_radius}" length="${wheel_width}"/>
+            </geometry>
+            <origin xyz="0.0 0.0 0.0" rpy="0.0 0.0 0.0"/>
         </collision>
         <inertial>
@@ -79,14 +80,15 @@
         <visual>
             <geometry>
-                <cylinder radius="${wheel_radius}" length="${wheel_width}"/>
-            </geometry>
-            <origin xyz="0.0 0.0 0.03" rpy="0.0 0.0 0.0"/>
-            <material name="grey"/>
-        </visual>
-        <collision>
-            <geometry>
-                <cylinder radius="${wheel_radius}" length="${wheel_width}"/>
-            </geometry>
-            <origin xyz="0.0 0.0 0.03" rpy="0.0 0.0 0.0"/>
+                <!--cylinder radius="${wheel_radius}" length="${wheel_width}"/-->
+                <mesh filename="file://$(find tf_broadcast_package)/meshes/Mecanum-Wheel-Left.STL" scale="0.001 0.001 0.001"/>
+            </geometry>
+            <origin xyz="-${wheel_radius} ${wheel_radius} ${wheel_width}" rpy="${pi} 0.0 0.0"/>
+            <material name="grey"/>
+        </visual>
+        <collision>
+            <geometry>
+                <cylinder radius="${wheel_radius}" length="${wheel_width}"/>
+            </geometry>
+            <origin xyz="0.0 0.0 0.0" rpy="0.0 0.0 0.0"/>
         </collision>
         <inertial>
@@ -99,18 +101,19 @@
         <visual>
             <geometry>
-                <cylinder radius="${wheel_radius}" length="${wheel_width}"/>
-            </geometry>
-            <origin xyz="0.0 0.0 0.03" rpy="0.0 0.0 0.0"/>
-            <material name="grey"/>
-        </visual>
-        <collision>
-            <geometry>
-                <cylinder radius="${wheel_radius}" length="${wheel_width}"/>
-            </geometry>
-            <origin xyz="0.0 0.0 0.03" rpy="0.0 0.0 0.0"/>
-        </collision>
-        <inertial>
-            <mass value="1.0"/>
-            <origin xyz="0.0 0.0 0.0" rpy="0.0 0.0 0.0"/>
+                <!--cylinder radius="${wheel_radius}" length="${wheel_width}"/-->
+                <mesh filename="file://$(find tf_broadcast_package)/meshes/Mecanum-Wheel-Right.STL" scale="0.001 0.001 0.001"/>
+            </geometry>
+            <origin xyz="0.0 0.0 0.0" rpy="0.0 0.0 0.0"/>
+            <material name="grey"/>
+        </visual>
+        <collision>
+            <geometry>
+                <cylinder radius="${wheel_radius}" length="${wheel_width}"/>
+            </geometry>
+            <origin xyz="0.0 0.0 0.0" rpy="0.0 0.0 0.0"/>
+        </collision>
+        <inertial>
+            <mass value="1.0"/>
+            <origin xyz="0.0 0.0 0.03" rpy="0.0 0.0 0.0"/>
             <inertia ixx="0.1" ixy="0.0" ixz="0.0" iyy="0.1" iyz="0.0" izz="0.1"/>
         </inertial>
@@ -119,7 +122,7 @@
         <visual>
             <geometry>
-                <cylinder radius="0.05" length="0.05"/>
-            </geometry>
-            <origin xyz="0.0 0.0 0.0" rpy="0.0 0.0 0.0"/>
+                <mesh filename="file://$(find tf_broadcast_package)/meshes/RP-LiDAR.STL" scale="0.001 0.001 0.001"/>
+            </geometry>
+            <origin xyz="0.0 0.0 0.042" rpy="-${pi / 2} 0.0 ${pi}"/>
             <material name="red"/>
         </visual>
@@ -177,9 +180,4 @@
         </inertial>
     </link>
-    <!--joint name="world_to_chassis_joint" type="fixed">
-        <parent link="world"/>
-        <child link="base_link"/>
-        <origin xyz="0.0 0.0 0.0" rpy="0.0 0.0 0.0"/>
-    </joint-->
     <joint name="wheel_front_left_joint" type="continuous">
         <parent link="base_link"/>
@@ -213,5 +211,5 @@
         <parent link="base_link"/>
         <child link="lidar_link"/>
-        <origin xyz="0.0 -0.05 ${chassis_height}" rpy="${pi} 0.0 ${pi * 3 / 2}"/>
+        <origin xyz="0.062 0.05 ${chassis_height + lidar_height}" rpy="${pi} 0.0 ${pi * 3/ 2}"/>
     </joint>
     <joint name="camera_joint" type="fixed">

Commit message: fixed right wheels

File: src/tf_broadcast_package/urdf/roboost_mecanum_robot.urdf.xacro (robot description, xacro)
@@ -41,5 +41,5 @@
                 <mesh filename="file://$(find tf_broadcast_package)/meshes/Mecanum-Wheel-Left.STL" scale="0.001 0.001 0.001"/>
             </geometry>
-            <origin xyz="-${wheel_radius} ${wheel_radius} ${wheel_width}" rpy="${pi} 0.0 0.0"/>
+            <origin xyz="0.0 0.0 0.0" rpy="0.0 0.0 0.0"/>
             <material name="grey"/>
         </visual>
@@ -83,5 +83,5 @@
                 <mesh filename="file://$(find tf_broadcast_package)/meshes/Mecanum-Wheel-Left.STL" scale="0.001 0.001 0.001"/>
             </geometry>
-            <origin xyz="-${wheel_radius} ${wheel_radius} ${wheel_width}" rpy="${pi} 0.0 0.0"/>
+            <origin xyz="0.0 0.0 0.0" rpy="0.0 0.0 0.0"/>
             <material name="grey"/>
         </visual>
