Commit message: added joystick node

File: src/roboost/urdf/roboost_mecanum_robot.urdf.xacro (robot description, xacro)
@@ -8,5 +8,5 @@
     <xacro:property name="chassis_mass" value="20.0"/>
     <xacro:property name="chassis_inertia" value="4.0"/>
-    <xacro:property name="wheel_radius" value="0.0835"/>
+    <xacro:property name="wheel_radius" value="0.075"/> <!-- ! This is only the wheel redius for the simulated robot. Actual Radius might differ-->
     <xacro:property name="wheel_width" value="0.05"/>
     <xacro:property name="wheel_mass" value="1.0"/>
@@ -16,7 +16,11 @@
     <xacro:property name="track" value="0.38"/>
     <link name="base_link">
-        <visual>
-            <geometry>
-                <mesh filename="file://$(find tf_broadcast_package)/meshes/Chassis.STL" scale="0.001 0.001 0.001"/>
+    </link>
+    <link name="base_footprint">
+    </link>
+    <link name="chassis_link">
+        <visual>
+            <geometry>
+                <mesh filename="file://$(find roboost)/meshes/Chassis.STL" scale="0.001 0.001 0.001"/>
             </geometry>
             <origin xyz="0.0 0.0 0.0" rpy="${pi / 2} 0.0 0.0"/>
@@ -39,5 +43,5 @@
             <geometry>
                 <!--cylinder radius="${wheel_radius}" length="${wheel_width}"/-->
-                <mesh filename="file://$(find tf_broadcast_package)/meshes/Mecanum-Wheel-Left.STL" scale="0.001 0.001 0.001"/>
+                <mesh filename="file://$(find roboost)/meshes/Mecanum-Wheel-Left.STL" scale="0.001 0.001 0.001"/>
             </geometry>
             <origin xyz="0.0 0.0 0.0" rpy="0.0 0.0 0.0"/>
@@ -60,5 +64,5 @@
             <geometry>
                 <!--cylinder radius="${wheel_radius}" length="${wheel_width}"/-->
-                <mesh filename="file://$(find tf_broadcast_package)/meshes/Mecanum-Wheel-Right.STL" scale="0.001 0.001 0.001"/>
+                <mesh filename="file://$(find roboost)/meshes/Mecanum-Wheel-Right.STL" scale="0.001 0.001 0.001"/>
             </geometry>
             <origin xyz="0.0 0.0 0.0" rpy="0.0 0.0 0.0"/>
@@ -81,5 +85,5 @@
             <geometry>
                 <!--cylinder radius="${wheel_radius}" length="${wheel_width}"/-->
-                <mesh filename="file://$(find tf_broadcast_package)/meshes/Mecanum-Wheel-Left.STL" scale="0.001 0.001 0.001"/>
+                <mesh filename="file://$(find roboost)/meshes/Mecanum-Wheel-Left.STL" scale="0.001 0.001 0.001"/>
             </geometry>
             <origin xyz="0.0 0.0 0.0" rpy="0.0 0.0 0.0"/>
@@ -101,6 +105,5 @@
         <visual>
             <geometry>
-                <!--cylinder radius="${wheel_radius}" length="${wheel_width}"/-->
-                <mesh filename="file://$(find tf_broadcast_package)/meshes/Mecanum-Wheel-Right.STL" scale="0.001 0.001 0.001"/>
+                <mesh filename="file://$(find roboost)/meshes/Mecanum-Wheel-Right.STL" scale="0.001 0.001 0.001"/>
             </geometry>
             <origin xyz="0.0 0.0 0.0" rpy="0.0 0.0 0.0"/>
@@ -122,5 +125,5 @@
         <visual>
             <geometry>
-                <mesh filename="file://$(find tf_broadcast_package)/meshes/RP-LiDAR.STL" scale="0.001 0.001 0.001"/>
+                <mesh filename="file://$(find roboost)/meshes/RP-LiDAR.STL" scale="0.001 0.001 0.001"/>
             </geometry>
             <origin xyz="0.0 0.0 0.042" rpy="-${pi / 2} 0.0 ${pi}"/>
@@ -160,5 +163,5 @@
         </inertial>
     </link>
-    <link name="imu">
+    <link name="imu_link">
         <visual>
             <geometry>
@@ -180,6 +183,16 @@
         </inertial>
     </link>
+    <joint name="base_footprint_joint" type="fixed">
+        <parent link="base_footprint"/>
+        <child link="base_link"/>
+        <origin xyz="0.0 0.0 0.0" rpy="0.0 0.0 0.0"/>
+    </joint>
+    <joint name="chassis_joint" type="fixed">
+        <parent link="base_link"/>
+        <child link="chassis_link"/>
+        <origin xyz="0.0 0.0 ${wheel_radius}" rpy="0.0 0.0 0.0"/>
+    </joint>
     <joint name="wheel_front_left_joint" type="continuous">
-        <parent link="base_link"/>
+        <parent link="chassis_link"/>
         <child link="wheel_front_left_link"/>
         <origin xyz="${wheelbase / 2} ${track / 2} 0.0" rpy="${pi * 3 / 2} 0.0 0.0"/>
@@ -188,5 +201,5 @@
     </joint>
     <joint name="wheel_front_right_joint" type="continuous">
-        <parent link="base_link"/>
+        <parent link="chassis_link"/>
         <child link="wheel_front_right_link"/>
         <origin xyz="${wheelbase / 2} -${track / 2} 0.0" rpy="${pi / 2} 0.0 0.0"/>
@@ -195,5 +208,5 @@
     </joint>
     <joint name="wheel_back_left_joint" type="continuous">
-        <parent link="base_link"/>
+        <parent link="chassis_link"/>
         <child link="wheel_back_left_link"/>
         <origin xyz="-${wheelbase / 2} ${track / 2} 0.0" rpy="${pi * 3 / 2} 0.0 0.0"/>
@@ -202,5 +215,5 @@
     </joint>
     <joint name="wheel_back_right_joint" type="continuous">
-        <parent link="base_link"/>
+        <parent link="chassis_link"/>
         <child link="wheel_back_right_link"/>
         <origin xyz="-${wheelbase / 2} -${track / 2} 0.0" rpy="${pi / 2} 0.0 0.0"/>
@@ -209,16 +222,16 @@
     </joint>
     <joint name="lidar_joint" type="fixed">
-        <parent link="base_link"/>
+        <parent link="chassis_link"/>
         <child link="lidar_link"/>
         <origin xyz="0.062 0.05 ${chassis_height + lidar_height}" rpy="${pi} 0.0 ${pi * 3/ 2}"/>
     </joint>
     <joint name="camera_joint" type="fixed">
-        <parent link="base_link"/>
+        <parent link="chassis_link"/>
         <child link="camera_link"/>
         <origin xyz="${-chassis_length / 2} 0.08 ${chassis_height -0.05}" rpy="0.0 ${pi * 3 / 2} 0.0"/>
     </joint>
     <joint name="imu_joint" type="fixed">
-        <parent link="base_link"/>
-        <child link="imu"/>
+        <parent link="chassis_link"/>
+        <child link="imu_link"/>
         <origin xyz="${-chassis_length / 2 + 0.05} 0.08 ${chassis_height -0.015}" rpy="0.0 0.0 0.0"/>
     </joint>

Commit message: added mecanum gazebo simulation

File: src/roboost/urdf/roboost_mecanum_robot.urdf.xacro (robot description, xacro)
@@ -2,4 +2,21 @@
 <robot xmlns:xacro="http://www.ros.org/wiki/xacro"  name="roboost_mecanum_robot">
     <xacro:include filename="roboost_materials.xacro"/>
+    <!-- Simple Macro to calculate inertia -->
+    <xacro:macro name="cylinder_inertia" params="mass radius length">
+        <inertia ixx="${mass * (3 * radius * radius + length * length) / 12}"
+                 ixy="0.0"
+                 ixz="0.0"
+                 iyy="${mass * (3 * radius * radius + length * length) / 12}"
+                 iyz="0.0"
+                 izz="${mass * radius * radius / 2}"/>
+    </xacro:macro>
+    <xacro:macro name="box_inertia" params="mass x y z">
+        <inertia ixx="${mass * (y * y + z * z) / 12}"
+                 ixy="0.0"
+                 ixz="0.0"
+                 iyy="${mass * (x * x + z * z) / 12}"
+                 iyz="0.0"
+                 izz="${mass * (x * x + y * y) / 12}"/>
+    </xacro:macro>
     <!-- TODO: determine values -->
     <xacro:property name="chassis_length" value="0.42"/>
@@ -7,9 +24,7 @@
     <xacro:property name="chassis_height" value="0.108"/> <!-- ! Measured from wheel axis to top plate -->
     <xacro:property name="chassis_mass" value="20.0"/>
-    <xacro:property name="chassis_inertia" value="4.0"/>
     <xacro:property name="wheel_radius" value="0.075"/> <!-- ! This is only the wheel redius for the simulated robot. Actual Radius might differ-->
     <xacro:property name="wheel_width" value="0.05"/>
     <xacro:property name="wheel_mass" value="1.0"/>
-    <xacro:property name="wheel_inertia" value="0.1"/>
     <xacro:property name="lidar_height" value="0.0575"/>
     <xacro:property name="wheelbase" value="0.3185"/>
@@ -36,7 +51,10 @@
             <mass value="${chassis_mass}"/>
             <origin xyz="0.0 0.0 ${chassis_height / 2}" rpy="0.0 0.0 0.0"/>
-            <inertia ixx="${chassis_inertia}" ixy="0.0" ixz="0.0" iyy="${chassis_inertia}" iyz="0.0" izz="${chassis_inertia}"/>
-        </inertial>
-    </link>
+            <xacro:box_inertia mass="${chassis_mass}" x="${chassis_length}" y="${chassis_width}" z="${chassis_height}"/>
+        </inertial>
+    </link>
+    <gazebo reference="chassis_link">
+        <material>Gazebo/Orange</material>
+    </gazebo>
     <link name="wheel_front_left_link">
         <visual>
@@ -57,7 +75,16 @@
             <mass value="1.0"/>
             <origin xyz="0.0 0.0 0.03" rpy="0.0 0.0 0.0"/>
-            <inertia ixx="0.1" ixy="0.0" ixz="0.0" iyy="0.1" iyz="0.0" izz="0.1"/>
-        </inertial>
-    </link>
+            <xacro:cylinder_inertia mass="${wheel_mass}" radius="${wheel_radius}" length="${wheel_width}"/>
+        </inertial>
+    </link>
+    <gazebo reference="wheel_front_left_link">
+        <material>Gazebo/Grey</material>
+        <mu1 value="1.0"/>
+        <mu2 value="1.0"/>
+        <kp value="1000000.0"/>
+        <kd value="1.0"/>
+        <fdir1 value="1 0 0"/>
+        <turnGravityOff>false</turnGravityOff>
+    </gazebo>
     <link name="wheel_front_right_link">
         <visual>
@@ -78,7 +105,16 @@
             <mass value="1.0"/>
             <origin xyz="0.0 0.0 0.03" rpy="0.0 0.0 0.0"/>
-            <inertia ixx="0.1" ixy="0.0" ixz="0.0" iyy="0.1" iyz="0.0" izz="0.1"/>
-        </inertial>
-    </link>
+            <xacro:cylinder_inertia mass="${wheel_mass}" radius="${wheel_radius}" length="${wheel_width}"/>
+        </inertial>
+    </link>
+    <gazebo reference="wheel_front_right_link">
+        <material>Gazebo/Grey</material>
+        <mu1 value="1.0"/>
+        <mu2 value="1.0"/>
+        <kp value="1000000.0"/>
+        <kd value="1.0"/>
+        <fdir1 value="1 0 0"/>
+        <turnGravityOff>false</turnGravityOff>
+    </gazebo>
     <link name="wheel_back_left_link">
         <visual>
@@ -99,7 +135,16 @@
             <mass value="1.0"/>
             <origin xyz="0.0 0.0 0.03" rpy="0.0 0.0 0.0"/>
-            <inertia ixx="0.1" ixy="0.0" ixz="0.0" iyy="0.1" iyz="0.0" izz="0.1"/>
-        </inertial>
-    </link>
+            <xacro:cylinder_inertia mass="${wheel_mass}" radius="${wheel_radius}" length="${wheel_width}"/>
+        </inertial>
+    </link>
+    <gazebo reference="wheel_back_left_link">
+        <material>Gazebo/Grey</material>
+        <mu1 value="1.0"/>
+        <mu2 value="1.0"/>
+        <kp value="1000000.0"/>
+        <kd value="1.0"/>
+        <fdir1 value="1 0 0"/>
+        <turnGravityOff>false</turnGravityOff>
+    </gazebo>
     <link name="wheel_back_right_link">
         <visual>
@@ -119,7 +164,16 @@
             <mass value="1.0"/>
             <origin xyz="0.0 0.0 0.03" rpy="0.0 0.0 0.0"/>
-            <inertia ixx="0.1" ixy="0.0" ixz="0.0" iyy="0.1" iyz="0.0" izz="0.1"/>
-        </inertial>
-    </link>
+            <xacro:cylinder_inertia mass="${wheel_mass}" radius="${wheel_radius}" length="${wheel_width}"/>
+        </inertial>
+    </link>
+    <gazebo reference="wheel_back_right_link">
+        <material>Gazebo/Grey</material>
+        <mu1 value="1.0"/>
+        <mu2 value="1.0"/>
+        <kp value="1000000.0"/>
+        <kd value="1.0"/>
+        <fdir1 value="1 0 0"/>
+        <turnGravityOff>false</turnGravityOff>
+    </gazebo>
     <link name="lidar_link">
         <visual>
@@ -139,7 +193,10 @@
             <mass value="1.0"/>
             <origin xyz="0.0 0.0 0.0" rpy="0.0 0.0 0.0"/>
-            <inertia ixx="0.1" ixy="0.0" ixz="0.0" iyy="0.1" iyz="0.0" izz="0.1"/>
-        </inertial>
-    </link>
+            <xacro:cylinder_inertia mass="${wheel_mass}" radius="${wheel_radius}" length="${wheel_width}"/>
+        </inertial>
+    </link>
+    <gazebo reference="lidar_link">
+        <material>Gazebo/Red</material>
+    </gazebo>
     <link name="camera_link">
         <visual>
@@ -151,16 +208,8 @@
             <material name="purple"/>
         </visual>
-        <collision>
-            <geometry>
-                <box size="0.02 0.02 0.02"/>
-            </geometry>
-            <origin xyz="0.0 0.0 0.0" rpy="0.0 0.0 0.0"/>
-        </collision>
-        <inertial>
-            <mass value="1.0"/>
-            <origin xyz="0.0 0.0 0.0" rpy="0.0 0.0 0.0"/>
-            <inertia ixx="0.01" ixy="0.0" ixz="0.0" iyy="0.01" iyz="0.0" izz="0.01"/>
-        </inertial>
-    </link>
+    </link>
+    <gazebo reference="camera_link">
+        <material>Gazebo/Purple</material>
+    </gazebo>
     <link name="imu_link">
         <visual>
@@ -171,21 +220,8 @@
             <material name="blue"/>
         </visual>
-        <collision>
-            <geometry>
-                <box size="0.02 0.02 0.01"/>
-            </geometry>
-            <origin xyz="0.0 0.0 0.0" rpy="0.0 0.0 0.0"/>
-        </collision>
-        <inertial>
-            <mass value="1.0"/>
-            <origin xyz="0.0 0.0 0.0" rpy="0.0 0.0 0.0"/>
-            <inertia ixx="0.01" ixy="0.0" ixz="0.0" iyy="0.01" iyz="0.0" izz="0.01"/>
-        </inertial>
-    </link>
-    <joint name="base_footprint_joint" type="fixed">
-        <parent link="base_footprint"/>
-        <child link="base_link"/>
-        <origin xyz="0.0 0.0 0.0" rpy="0.0 0.0 0.0"/>
-    </joint>
+    </link>
+    <gazebo reference="imu_link">
+        <material>Gazebo/Blue</material>
+    </gazebo>
     <joint name="chassis_joint" type="fixed">
         <parent link="base_link"/>
@@ -193,4 +229,9 @@
         <origin xyz="0.0 0.0 ${wheel_radius}" rpy="0.0 0.0 0.0"/>
     </joint>
+    <joint name="base_footprint_joint" type="fixed">
+        <parent link="base_link"/>
+        <child link="base_footprint"/>
+        <origin xyz="0.0 0.0 -${wheel_radius}" rpy="0.0 0.0 0.0"/>
+    </joint>
     <joint name="wheel_front_left_joint" type="continuous">
         <parent link="chassis_link"/>
@@ -198,5 +239,6 @@
         <origin xyz="${wheelbase / 2} ${track / 2} 0.0" rpy="${pi * 3 / 2} 0.0 0.0"/>
         <axis xyz="0.0 0.0 1.0"/>
-        <limit effort="1000.0" velocity="1000.0"/>
+        <limit effort="100.0" velocity="100.0"/>
+        <joint_properties damping="0.0" friction="0.0"/>
     </joint>
     <joint name="wheel_front_right_joint" type="continuous">
@@ -205,5 +247,6 @@
         <origin xyz="${wheelbase / 2} -${track / 2} 0.0" rpy="${pi / 2} 0.0 0.0"/>
         <axis xyz="0.0 0.0 1.0"/>
-        <limit effort="1000.0" velocity="1000.0"/>
+        <limit effort="100.0" velocity="100.0"/>
+        <joint_properties damping="0.0" friction="0.0"/>
     </joint>
     <joint name="wheel_back_left_joint" type="continuous">
@@ -212,5 +255,6 @@
         <origin xyz="-${wheelbase / 2} ${track / 2} 0.0" rpy="${pi * 3 / 2} 0.0 0.0"/>
         <axis xyz="0.0 0.0 1.0"/>
-        <limit effort="1000.0" velocity="1000.0"/>
+        <limit effort="100.0" velocity="100.0"/>
+        <joint_properties damping="0.0" friction="0.0"/>
     </joint>
     <joint name="wheel_back_right_joint" type="continuous">
@@ -219,5 +263,6 @@
         <origin xyz="-${wheelbase / 2} -${track / 2} 0.0" rpy="${pi / 2} 0.0 0.0"/>
         <axis xyz="0.0 0.0 1.0"/>
-        <limit effort="1000.0" velocity="1000.0"/>
+        <limit effort="100.0" velocity="100.0"/>
+        <joint_properties damping="0.0" friction="0.0"/>
     </joint>
     <joint name="lidar_joint" type="fixed">
@@ -236,3 +281,44 @@
         <origin xyz="${-chassis_length / 2 + 0.05} 0.08 ${chassis_height -0.015}" rpy="0.0 0.0 0.0"/>
     </joint>
+    <transmission name="transmission_front_left">
+        <type>transmission_interface/SimpleTransmission</type>
+        <joint name="wheel_front_left_joint">
+            <hardwareInterface>hardware_interface/EffortJointInterface</hardwareInterface>
+        </joint>
+        <actuator name="front_left_motor">
+            <hardwareInterface>hardware_interface/EffortJointInterface</hardwareInterface>
+            <mechanicalReduction>1</mechanicalReduction>
+        </actuator>
+    </transmission>
+    <transmission name="transmission_front_right">
+        <type>transmission_interface/SimpleTransmission</type>
+        <joint name="wheel_front_right_joint">
+            <hardwareInterface>hardware_interface/EffortJointInterface</hardwareInterface>
+        </joint>
+        <actuator name="front_right_motor">
+            <hardwareInterface>hardware_interface/EffortJointInterface</hardwareInterface>
+            <mechanicalReduction>1</mechanicalReduction>
+        </actuator>
+    </transmission>
+    <transmission name="transmission_back_left">
+        <type>transmission_interface/SimpleTransmission</type>
+        <joint name="wheel_back_left_joint">
+            <hardwareInterface>hardware_interface/EffortJointInterface</hardwareInterface>
+        </joint>
+        <actuator name="back_left_motor">
+            <hardwareInterface>hardware_interface/EffortJointInterface</hardwareInterface>
+            <mechanicalReduction>1</mechanicalReduction>
+        </actuator>
+    </transmission>
+    <transmission name="transmission_back_right">
+        <type>transmission_interface/SimpleTransmission</type>
+        <joint name="wheel_back_right_joint">
+            <hardwareInterface>hardware_interface/EffortJointInterface</hardwareInterface>
+        </joint>
+        <actuator name="back_right_motor">
+            <hardwareInterface>hardware_interface/EffortJointInterface</hardwareInterface>
+            <mechanicalReduction>1</mechanicalReduction>
+        </actuator>
+    </transmission>
+    <xacro:include filename="gazebo_control.xacro"/>
 </robot>
