Commit message: created home_map; added amcl support

File: src/roboost/robot_descriptions/robots/mecanum_robot.urdf.xacro (robot description, xacro)
@@ -40,5 +40,5 @@
     <!-- Sensors -->
     <xacro:lidar name="lidar" parent="chassis_link">
-        <origin xyz="0.062 0.05 ${chassis_height + lidar_height}" rpy="${pi} 0.0 ${pi * 3/ 2}"/>
+        <origin xyz="0.057 0.045 ${chassis_height + lidar_height}" rpy="${pi} 0.0 ${pi * 3/ 2}"/>
     </xacro:lidar>
     <xacro:camera name="camera" parent="chassis_link">

Commit message: added instructions for Nav2

File: src/roboost/robot_descriptions/robots/mecanum_robot.urdf.xacro (robot description, xacro)
@@ -16,5 +16,5 @@
     <!-- Base Footprint link-->
     <link name="base_footprint"/>
-    <joint name="base_footprint_joint" type="fixed">
+    <joint name="base_joint" type="fixed">
         <parent link="base_link"/>
         <child link="base_footprint"/>
